File: G15_Diode_1/G15_Diode_1.kicad_pcb (KiCad board)
At the start: 2 copper layers, 92.1 x 103.6 mm, 17 parts, among them J1 Conn_02x18_Row_Letter_First

Commit message: Minor updates, and board files.
Routing:
- net /C_{8}: track 39.8 -> 79.6 mm
- net /C_{1}: track 22.0 -> 44.0 mm
- net /C_{5}: track 16.5 -> 33.1 mm
- net /C_{6}: track 16.4 -> 32.8 mm
- net /C_{7}: track 36.5 -> 39.6 mm
Changed lines of the file:
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@@
       (layerselection 0x00010fc_ffffffff)
       (disableapertmacros false)
-      (usegerberextensions false)
+      (usegerberextensions true)
       (usegerberattributes true)
       (usegerberadvancedattributes true)
@@
       (plotinvisibletext false)
       (sketchpadsonfab false)
-      (subtractmaskfromsilk false)
+      (subtractmaskfromsilk true)
       (outputformat 1)
       (mirror false)
-      (drillshape 1)
+      (drillshape 0)
       (scaleselection 1)
-      (outputdirectory "")
+      (outputdirectory "G15_Diode_1_Board_Files/")
     )
   )
@@
     (fp_line (start 4.83 -1.12) (end 4.83 1.12) (layer "F.SilkS") (width 0.12))
     (fp_line (start 4.23 -1.12) (end 4.23 1.12) (layer "F.SilkS") (width 0.12))
+    (fp_line (start -1.05 -1.25) (end -1.05 1.25) (layer "F.CrtYd") (width 0.05))
     (fp_line (start -1.05 1.25) (end 13.75 1.25) (layer "F.CrtYd") (width 0.05))
     (fp_line (start 13.75 -1.25) (end -1.05 -1.25) (layer "F.CrtYd") (width 0.05))
     (fp_line (start 13.75 1.25) (end 13.75 -1.25) (layer "F.CrtYd") (width 0.05))
-    (fp_line (start -1.05 -1.25) (end -1.05 1.25) (layer "F.CrtYd") (width 0.05))
     (fp_line (start 4.35 -1) (end 4.35 1) (layer "F.Fab") (width 0.1))
     (fp_line (start 0 0) (end 4.35 0) (layer "F.Fab") (width 0.1))
@@
   (segment (start 179.771875 149.793125) (end 183.515 136.525) (width 1.27) (layer "F.Cu") (net 2))
   (segment (start 179.771875 157.997625) (end 179.771875 149.793125) (width 1.27) (layer "F.Cu") (net 2))
+  (segment (start 179.771875 157.997625) (end 179.771875 149.793125) (width 1.27) (layer "B.Cu") (net 2))
+  (segment (start 179.771875 149.793125) (end 183.515 136.525) (width 1.27) (layer "B.Cu") (net 2))
   (segment (start 163.83 123.825) (end 158.75 123.825) (width 1.27) (layer "F.Cu") (net 3))
   (segment (start 158.75 123.825) (end 140.97 120.015) (width 1.27) (layer "F.Cu") (net 3))
@@
   (segment (start 132.146875 157.997625) (end 132.146875 154.238125) (width 1.27) (layer "F.Cu") (net 7))
   (segment (start 132.146875 154.238125) (end 133.985 141.605) (width 1.27) (layer "F.Cu") (net 7))
+  (segment (start 132.146875 154.238125) (end 133.985 141.605) (width 1.27) (layer "B.Cu") (net 7))
+  (segment (start 132.146875 157.997625) (end 132.146875 154.238125) (width 1.27) (layer "B.Cu") (net 7))
   (segment (start 150.277377 132.387421) (end 143.47544 127.986167) (width 1.27) (layer "F.Cu") (net 8))
   (segment (start 171.45 133.35) (end 171.834375 133.734375) (width 1.27) (layer "F.Cu") (net 8))
@@
   (segment (start 128.178125 154.396875) (end 128.905 141.605) (width 1.27) (layer "F.Cu") (net 9))
   (segment (start 128.178125 157.997625) (end 128.178125 154.396875) (width 1.27) (layer "F.Cu") (net 9))
+  (segment (start 128.178125 157.997625) (end 128.178125 154.396875) (width 1.27) (layer "B.Cu") (net 9))
+  (segment (start 128.178125 154.396875) (end 128.905 141.605) (width 1.27) (layer "B.Cu") (net 9))
   (segment (start 112.303125 151.038125) (end 111.76 150.495) (width 1.27) (layer "F.Cu") (net 10))
   (segment (start 112.303125 157.997625) (end 112.303125 151.038125) (width 1.27) (layer "F.Cu") (net 10))
   (via (at 111.76 150.495) (size 2) (drill 1.27) (layers "F.Cu" "B.Cu") (net 10))
-  (segment (start 117.229552 143.80612) (end 119.238766 138.783085) (width 1.27) (layer "B.Cu") (net 10))
-  (segment (start 119.564683 138.097571) (end 122.555 132.715) (width 1.27) (layer "B.Cu") (net 10))
-  (segment (start 111.76 150.495) (end 116.143148 145.563959) (width 1.27) (layer "B.Cu") (net 10))
+  (segment (start 117.199223 133.538966) (end 122.555 132.715) (width 1.27) (layer "B.Cu") (net 10))
   (segment (start 112.303125 157.997625) (end 112.303125 151.038125) (width 1.27) (layer "B.Cu") (net 10))
+  (segment (start 111.76 150.495) (end 113.853966 136.884223) (width 1.27) (layer "B.Cu") (net 10))
   (segment (start 112.303125 151.038125) (end 111.76 150.495) (width 1.27) (layer "B.Cu") (net 10))
-  (arc (start 119.564683 138.097571) (mid 119.390873 138.435169) (end 119.238766 138.783085) (width 1.27) (layer "B.Cu") (net 10))
-  (arc (start 117.229552 143.80612) (mid 116.762597 144.732163) (end 116.143148 145.563959) (width 1.27) (layer "B.Cu") (net 10))
+  (arc (start 117.199223 133.538966) (mid 114.979025 134.664025) (end 113.853966 136.884223) (width 1.27) (layer "B.Cu") (net 10))
   (segment (start 148.021875 157.997625) (end 148.021875 147.386875) (width 1.27) (layer "F.Cu") (net 11))
   (segment (start 148.021875 147.386875) (end 147.955 147.32) (width 1.27) (layer "F.Cu") (net 11))
@@
   (arc (start 137.01811 143.386061) (mid 136.90534 141.659259) (end 136.304433 140.036461) (width 1.27) (layer "F.Cu") (net 12))
   (arc (start 129.331781 135.083641) (mid 132.781077 135.717385) (end 135.286899 138.170981) (width 1.27) (layer "F.Cu") (net 12))
+  (segment (start 129.331781 135.083641) (end 116.84 136.525) (width 1.27) (layer "B.Cu") (net 12))
+  (segment (start 136.115625 157.997625) (end 136.115625 154.714375) (width 1.27) (layer "B.Cu") (net 12))
+  (segment (start 136.115625 154.714375) (end 137.01811 143.386061) (width 1.27) (layer "B.Cu") (net 12))
+  (segment (start 136.304433 140.036461) (end 135.286899 138.170981) (width 1.27) (layer "B.Cu") (net 12))
+  (arc (start 137.01811 143.386061) (mid 136.90534 141.659259) (end 136.304433 140.036461) (width 1.27) (layer "B.Cu") (net 12))
+  (arc (start 129.331781 135.083641) (mid 132.781077 135.717385) (end 135.286899 138.170981) (width 1.27) (layer "B.Cu") (net 12))
   (segment (start 144.053125 157.997625) (end 144.053125 143.601875) (width 1.27) (layer "F.Cu") (net 13))
   (segment (start 144.053125 143.601875) (end 144.145 143.51) (width 1.27) (layer "F.Cu") (net 13))
