File: G15_Diode_Clamp/G15_Diode_Clamp.kicad_pcb (KiCad board)
At the start: 2 copper layers, 92.1 x 103.6 mm, 39 parts, among them J1 Conn_02x18_Row_Letter_First

Commit message: Minor updates, and board files.
Routing:
- net /+100V: track 127.7 -> 145.4 mm, vias 0 -> 1
- net /CL_{12}: track 87.0 -> 104.3 mm
- net /CL_{1}: track 87.0 -> 103.9 mm
- net /CL_{5}: track 86.1 -> 102.3 mm
- net /CL_{8}: track 85.5 -> 101.1 mm
- net /CL_{6}: track 88.5 -> 104.0 mm
- net /CL_{7}: track 87.7 -> 102.3 mm
- net /CL_{10}: track 84.4 -> 98.9 mm
- net /CL_{3}: track 84.4 -> 98.7 mm
- net GND: track 148.5 -> 161.6 mm, vias 0 -> 1
- net /CL_{11}: track 85.5 -> 98.0 mm
- net /CL_{4}: track 85.0 -> 97.1 mm
- net /CL_{2}: track 85.1 -> 97.0 mm
- net /CL_{9}: track 84.6 -> 96.2 mm
- net /-20V: track 257.9 -> 269.3 mm, vias 0 -> 1
