File: G15_Green_RA/G15_Green_RA.kicad_pcb (KiCad board)
At the start: 2 copper layers, 92.1 x 88.9 mm, 43 parts, among them J1 Conn_02x18_Row_Letter_First, T1 1:4

Commit message: Update Green Read Amp
Parts:
- turned TP1 to 180 degrees
- turned TP10 to 180 degrees
- turned TP11 to 180 degrees
- turned TP12 to 180 degrees
- turned TP13 to 180 degrees
- turned TP14 to 180 degrees
- turned TP15 to 180 degrees
- turned TP2 to 180 degrees
- turned TP3 to 180 degrees
- turned TP4 to 180 degrees
- turned TP5 to 180 degrees
- turned TP6 to 180 degrees
- turned TP7 to 180 degrees
- turned TP8 to 180 degrees
- turned TP9 to 180 degrees
